File: LiamsWork/VoltageRegulator/PCBDesignFiles/VoltageRegulator/VoltageSourcePCBLT6000.sch (EAGLE design)
At the start: 23 parts, among them U1 LT1494S8

Commit message: Files updated to contain recent developments, added Amplifier power supply file
Parts:
- added C4: 0.01u, capacitor-wima:C5/2.5
- added C5: 10u, capacitor-wima:C5/2.5
- added D4, D5, D6, D7, D8, D9: (no value), semicon-smd-ipc:D-SOD123
- added R10: 309k, SparkFun-Resistors:RESISTOR0805
- added R8: 10M, SparkFun-Resistors:RESISTOR0805
- C1: value 10nF -> 0.01u
- R5: value 6.81M -> 10M
- R9: value 499k -> 2M
- U1: value LT1494S8 -> LT6000DCB; device RequiredComponents:LT1494S8 -> RequiredComponents:LT6000DCB
- renumbered SWITCHDPDT to DPDTVOLT, SWITCHDPST to DPDTONOFF
Connections:
- net N$9 renamed IN+
- removed net N$13: R9.1, U1.IN-, VR2.CW, VR2.WIPER
- removed net N$3: D2.ANODE, LEDCIRCUIT-2.KL, U1.V-
- new net IN-: R10.1, U1.IN-, VR2.CW, VR2.WIPER
- new net N$14: BATTERY-1.KL, C1.1, D4.A, LEDCIRCUIT-1.KL
- new net N$15: R5.1, R8.1, R9.2
- new net N$9: D7.A, D8.C
- new net OUT: R3.1, R5.2, R8.2, U1.OUT
- new net V+: C4.1, C5.1, DPDTONOFF-1.KL, R1.2, U1.V+
- new net V-: C4.2, C5.2, D2.ANODE, D9.A, U1.V-
- net N$1: now also BATTERY-2.KL, C1.2, D7.C, LEDCIRCUIT-2.KL; no longer BATTERY-1.KL, C1.1
- net N$10: now also D8.A, D9.C; no longer R3.1, R5.2, U1.OUT
- net N$2: now also D6.C, DPDTONOFF-2.KL; no longer BATTERY-2.KL, C1.2
- net N$20: now also R10.2, R9.1; no longer R5.1, R9.2
- net N$4: now also D4.C, D5.A; no longer DPDTONOFF-2.KL, LEDCIRCUIT-1.KL
- net N$5: now also D5.C, D6.A; no longer DPDTONOFF-1.KL, R1.2, U1.V+
Other:
- moved on the sheet: BATTERY-1, BATTERY-2, C1, LEDCIRCUIT-1, LEDCIRCUIT-2, R4, R5, R9, U1, VR2
